Commit message: update the rover urdf and simulation

File: src/meer_description/urdf/gazebo_plugins.xacro (robot description, xacro)
@@ -22,7 +22,7 @@
       <right_joint>front_right_wheel</right_joint>
       <right_joint>back_right_wheel</right_joint>
-      <!-- Kinematics -->
-      <wheel_separation>0.61</wheel_separation>
-      <wheel_radius>0.10</wheel_radius>
+      <!-- Kinematics from Real CAD Model -->
+      <wheel_separation>0.8184</wheel_separation>
+      <wheel_radius>0.1155</wheel_radius>
       <!-- Topics -->
       <topic>/cmd_vel</topic>
@@ -53,6 +53,4 @@
       <joint_name>front_right_wheel</joint_name>
       <joint_name>back_right_wheel</joint_name>
-      <joint_name>leftrocker</joint_name>
-      <joint_name>rightrcker</joint_name>
     </plugin>
   </gazebo>
@@ -61,5 +59,5 @@
   <xacro:macro name="wheel_gazebo_friction" params="link_name">
     <gazebo reference="${link_name}">
-      <mu1>1.0</mu1>
+      <mu1>1.2</mu1>
       <mu2>0.4</mu2>
       <kp>1e6</kp>
@@ -78,4 +76,7 @@
   <gazebo reference="base_link">
     <material>Gazebo/DarkGrey</material>
+  </gazebo>
+  <gazebo reference="enclsr">
+    <material>Gazebo/Grey</material>
   </gazebo>
   <gazebo reference="Left_rocker">

File: src/meer_description/urdf/meer_rover.urdf.xacro (robot description, xacro)
@@ -8,4 +8,10 @@
     - Up       : +Z
     - Wheel axle rotation axis: +Y [0 1 0]
+  Integrated from Real Physical CAD Model (SW2URDF):
+    - Meshes: package://meer_description/meshes/*.STL
+    - Kinematics: 4WD Skid-Steer with twin articulated rocker suspension
+    - Wheel radius: 0.1155 m (115.5 mm)
+    - Wheel track separation: 0.8184 m (818.4 mm)
+    - Wheelbase: 0.682 m (682 mm)
 -->
 <robot name="meer_rover" xmlns:xacro="http://www.ros.org/wiki/xacro">
@@ -24,51 +30,86 @@
     <parent link="base_footprint"/>
     <child link="base_link"/>
-    <origin xyz="0.0 0.0 0.22" rpy="0 0 0"/>
+    <origin xyz="0.0 0.0 0.31074" rpy="0 0 0"/>
   </joint>
   <!-- =====================================================================
        BASE LINK (Chassis body)
-       Length (X): 0.65 m
-       Width  (Y): 0.45 m
-       Height (Z): 0.12 m
-       Mass: 2.778 kg
+       Real CAD Model bounds: Length (X)=0.8716 m, Width (Y)=0.3973 m, Height (Z)=0.3494 m
+       Mass: 2.7788 kg (from SolidWorks mass properties)
   ====================================================================== -->
   <link name="base_link">
     <visual>
-      <geometry>
-        <box size="0.65 0.45 0.12"/>
-      </geometry>
-      <origin xyz="0 0 0" rpy="0 0 0"/>
+      <origin xyz="0 0 0" rpy="0 0 -1.5707963"/>
+      <geometry>
+        <mesh filename="package://meer_description/meshes/base_link.STL"/>
+      </geometry>
       <material name="dark_grey"/>
     </visual>
     <collision>
-      <geometry>
-        <box size="0.65 0.45 0.12"/>
-      </geometry>
-      <origin xyz="0 0 0" rpy="0 0 0"/>
-    </collision>
-    <inertial>
-      <mass value="2.778"/>
-      <origin xyz="0 0 0" rpy="0 0 0"/>
-      <xacro:solid_box_inertia m="2.778" x="0.65" y="0.45" z="0.12"/>
-    </inertial>
-  </link>
-  <!-- =====================================================================
-       LEFT SUSPENSION CHAIN (Rocker + Wheels on +Y)
-  ====================================================================== -->
-  <!-- Left Bearing (fixed mount on left side of chassis at Y = +0.225) -->
+      <origin xyz="0.03 0.0 0.08" rpy="0 0 0"/>
+      <geometry>
+        <box size="0.87 0.40 0.25"/>
+      </geometry>
+    </collision>
+    <inertial>
+      <mass value="2.7788"/>
+      <origin xyz="-0.00219 0.00508 -0.00451" rpy="0 0 0"/>
+      <inertia
+        ixx="0.050189" ixy="0.0" ixz="0.026071"
+        iyy="0.196732" iyz="0.0" izz="0.227775"/>
+    </inertial>
+  </link>
+  <!-- =====================================================================
+       ENCLOSURE (Electronics housing mounted on top of base_link)
+       Real CAD Model bounds: Length (X)=0.7878 m, Width (Y)=0.4064 m, Height (Z)=0.1727 m
+  ====================================================================== -->
+  <link name="enclsr">
+    <visual>
+      <origin xyz="0 0 0" rpy="0 0 -1.5707963"/>
+      <geometry>
+        <mesh filename="package://meer_description/meshes/enclsr.STL"/>
+      </geometry>
+      <material name="silver"/>
+    </visual>
+    <collision>
+      <origin xyz="0.09 0.0 0.086" rpy="0 0 0"/>
+      <geometry>
+        <box size="0.78 0.40 0.17"/>
+      </geometry>
+    </collision>
+    <inertial>
+      <mass value="0.5"/>
+      <origin xyz="0.09 0.0 0.086" rpy="0 0 0"/>
+      <xacro:solid_box_inertia m="0.5" x="0.78" y="0.40" z="0.17"/>
+    </inertial>
+  </link>
+  <joint name="enclsr_joint" type="fixed">
+    <parent link="base_link"/>
+    <child link="enclsr"/>
+    <origin xyz="0 0 0" rpy="0 0 0"/>
+  </joint>
+  <!-- =====================================================================
+       LEFT SUSPENSION CHAIN (Bearing + Rocker + Wheels on +Y Left)
+  ====================================================================== -->
+  <!-- Left Bearing (fixed mount on left side of chassis at Y = +0.2237 m) -->
   <link name="left_bearing">
     <visual>
-      <geometry><cylinder radius="0.02" length="0.04"/></geometry>
+      <origin xyz="0 0 0" rpy="0 0 -1.5707963"/>
+      <geometry>
+        <mesh filename="package://meer_description/meshes/left_bearing.STL"/>
+      </geometry>
+      <material name="silver"/>
+    </visual>
+    <collision>
       <origin xyz="0 0 0" rpy="1.5707963 0 0"/>
-      <material name="silver"/>
-    </visual>
-    <collision>
-      <geometry><cylinder radius="0.02" length="0.04"/></geometry>
-      <origin xyz="0 0 0" rpy="1.5707963 0 0"/>
-    </collision>
-    <inertial>
-      <mass value="0.103"/>
-      <origin xyz="0 0 0" rpy="0 0 0"/>
-      <xacro:solid_cylinder_inertia m="0.103" r="0.02" h="0.04"/>
+      <geometry>
+        <cylinder radius="0.03" length="0.04"/>
+      </geometry>
+    </collision>
+    <inertial>
+      <mass value="0.1032"/>
+      <origin xyz="-0.00004 -0.03813 0.00793" rpy="0 0 0"/>
+      <inertia
+        ixx="0.000039" ixy="0.0" ixz="0.0"
+        iyy="0.000119" iyz="0.0" izz="0.000100"/>
     </inertial>
   </link>
@@ -76,46 +117,55 @@
     <parent link="base_link"/>
     <child link="left_bearing"/>
-    <origin xyz="0.0 0.225 -0.05" rpy="0 0 0"/>
-  </joint>
-  <!-- Left Rocker (revolute joint around pitch Y axis) -->
+    <origin xyz="0.0015 0.22373 -0.0586" rpy="0 0 0"/>
+  </joint>
+  <!-- Left Rocker (rigidly locked to chassis bearing, leveled with CAD compensation) -->
   <link name="Left_rocker">
     <visual>
-      <geometry><box size="0.60 0.05 0.04"/></geometry>
-      <origin xyz="0 0 0" rpy="0 0 0"/>
+      <origin xyz="0 0 0" rpy="0 0 -1.5707963"/>
+      <geometry>
+        <mesh filename="package://meer_description/meshes/Left_rocker.STL"/>
+      </geometry>
       <material name="orange"/>
     </visual>
     <collision>
-      <geometry><box size="0.60 0.05 0.04"/></geometry>
-      <origin xyz="0 0 0" rpy="0 0 0"/>
-    </collision>
-    <inertial>
-      <mass value="4.921"/>
-      <origin xyz="0 0 0" rpy="0 0 0"/>
-      <xacro:solid_box_inertia m="4.921" x="0.60" y="0.05" z="0.04"/>
-    </inertial>
-  </link>
-  <joint name="leftrocker" type="revolute">
+      <origin xyz="0.0 -0.05 -0.03" rpy="0 0 0"/>
+      <geometry>
+        <box size="0.72 0.05 0.05"/>
+      </geometry>
+    </collision>
+    <inertial>
+      <mass value="4.9215"/>
+      <origin xyz="-0.01847 0.00746 -0.00647" rpy="0 0 0"/>
+      <inertia
+        ixx="0.022827" ixy="0.000476" ixz="0.008313"
+        iyy="0.231464" iyz="0.000167" izz="0.214717"/>
+    </inertial>
+  </link>
+  <joint name="leftrocker" type="fixed">
     <parent link="left_bearing"/>
     <child link="Left_rocker"/>
-    <origin xyz="0 0.03 0" rpy="0 0 0"/>
-    <axis xyz="0 1 0"/>
-    <limit lower="-0.26" upper="0.26" effort="100" velocity="2.0"/>
-    <dynamics damping="0.5" friction="0.1"/>
-  </joint>
-  <!-- FLW — Front Left Wheel (continuous driven wheel, rolling around Y axis) -->
+    <origin xyz="0 0 0" rpy="0 0.03126 0"/>
+  </joint>
+  <!-- FLW — Front Left Wheel (driven wheel, rolling around Y axis) -->
   <link name="FLW">
     <visual>
-      <geometry><cylinder radius="0.10" length="0.07"/></geometry>
-      <origin xyz="0 0 0" rpy="1.5707963 0 0"/>
+      <origin xyz="0 0 0" rpy="0 0 -1.5707963"/>
+      <geometry>
+        <mesh filename="package://meer_description/meshes/FLW.STL"/>
+      </geometry>
       <material name="black"/>
     </visual>
     <collision>
-      <geometry><cylinder radius="0.10" length="0.07"/></geometry>
-      <origin xyz="0 0 0" rpy="1.5707963 0 0"/>
-    </collision>
-    <inertial>
-      <mass value="1.911"/>
-      <origin xyz="0 0 0" rpy="0 0 0"/>
-      <xacro:solid_cylinder_inertia m="1.911" r="0.10" h="0.07"/>
+      <origin xyz="0 -0.0444 0" rpy="1.5707963 0 0"/>
+      <geometry>
+        <cylinder radius="0.1155" length="0.0889"/>
+      </geometry>
+    </collision>
+    <inertial>
+      <mass value="1.9116"/>
+      <origin xyz="0.00004 -0.04682 0.0" rpy="0 0 0"/>
+      <inertia
+        ixx="0.005538" ixy="0.0" ixz="0.0"
+        iyy="0.008143" iyz="0.0" izz="0.005536"/>
     </inertial>
   </link>
@@ -123,24 +173,30 @@
     <parent link="Left_rocker"/>
     <child link="FLW"/>
-    <origin xyz="0.25 0.05 -0.07" rpy="0 0 0"/>
+    <origin xyz="0.34597 0.1908 -0.12589" rpy="0 0 0"/>
     <axis xyz="0 1 0"/>
     <limit effort="50" velocity="20"/>
-    <dynamics damping="0.1" friction="0.05"/>
-  </joint>
-  <!-- BLW — Back Left Wheel (continuous driven wheel, rolling around Y axis) -->
+    <dynamics damping="0.05" friction="0.02"/>
+  </joint>
+  <!-- BLW — Back Left Wheel (driven wheel, rolling around Y axis) -->
   <link name="BLW">
     <visual>
-      <geometry><cylinder radius="0.10" length="0.07"/></geometry>
-      <origin xyz="0 0 0" rpy="1.5707963 0 0"/>
+      <origin xyz="0 0 0" rpy="0 0 -1.5707963"/>
+      <geometry>
+        <mesh filename="package://meer_description/meshes/BLW.STL"/>
+      </geometry>
       <material name="black"/>
     </visual>
     <collision>
-      <geometry><cylinder radius="0.10" length="0.07"/></geometry>
-      <origin xyz="0 0 0" rpy="1.5707963 0 0"/>
-    </collision>
-    <inertial>
-      <mass value="1.911"/>
-      <origin xyz="0 0 0" rpy="0 0 0"/>
-      <xacro:solid_cylinder_inertia m="1.911" r="0.10" h="0.07"/>
+      <origin xyz="0 -0.0444 0" rpy="1.5707963 0 0"/>
+      <geometry>
+        <cylinder radius="0.1155" length="0.0889"/>
+      </geometry>
+    </collision>
+    <inertial>
+      <mass value="1.9116"/>
+      <origin xyz="0.00004 -0.04682 0.0" rpy="0 0 0"/>
+      <inertia
+        ixx="0.005538" ixy="0.0" ixz="0.0"
+        iyy="0.008143" iyz="0.0" izz="0.005536"/>
     </inertial>
   </link>
@@ -148,27 +204,33 @@
     <parent link="Left_rocker"/>
     <child link="BLW"/>
-    <origin xyz="-0.25 0.05 -0.07" rpy="0 0 0"/>
+    <origin xyz="-0.33792 0.1908 -0.14727" rpy="0 0 0"/>
     <axis xyz="0 1 0"/>
     <limit effort="50" velocity="20"/>
-    <dynamics damping="0.1" friction="0.05"/>
-  </joint>
-  <!-- =====================================================================
-       RIGHT SUSPENSION CHAIN (Rocker + Wheels on -Y)
-  ====================================================================== -->
-  <!-- Right Bearing (fixed mount on right side of chassis at Y = -0.225) -->
+    <dynamics damping="0.05" friction="0.02"/>
+  </joint>
+  <!-- =====================================================================
+       RIGHT SUSPENSION CHAIN (Bearing + Rocker + Wheels on -Y Right)
+  ====================================================================== -->
+  <!-- Right Bearing (fixed mount on right side of chassis at Y = -0.2130 m) -->
   <link name="right_bearing">
     <visual>
-      <geometry><cylinder radius="0.02" length="0.04"/></geometry>
+      <origin xyz="0 0 0" rpy="0 0 -1.5707963"/>
+      <geometry>
+        <mesh filename="package://meer_description/meshes/right_bearing.STL"/>
+      </geometry>
+      <material name="silver"/>
+    </visual>
+    <collision>
       <origin xyz="0 0 0" rpy="1.5707963 0 0"/>
-      <material name="silver"/>
-    </visual>
-    <collision>
-      <geometry><cylinder radius="0.02" length="0.04"/></geometry>
-      <origin xyz="0 0 0" rpy="1.5707963 0 0"/>
-    </collision>
-    <inertial>
-      <mass value="0.103"/>
-      <origin xyz="0 0 0" rpy="0 0 0"/>
-      <xacro:solid_cylinder_inertia m="0.103" r="0.02" h="0.04"/>
+      <geometry>
+        <cylinder radius="0.03" length="0.04"/>
+      </geometry>
+    </collision>
+    <inertial>
+      <mass value="0.1032"/>
+      <origin xyz="0.00004 0.03760 0.00793" rpy="0 0 0"/>
+      <inertia
+        ixx="0.000039" ixy="0.0" ixz="0.0"
+        iyy="0.000119" iyz="0.0" izz="0.000100"/>
     </inertial>
   </link>
@@ -176,46 +238,55 @@
     <parent link="base_link"/>
     <child link="right_bearing"/>
-    <origin xyz="0.0 -0.225 -0.05" rpy="0 0 0"/>
-  </joint>
-  <!-- Right Rocker (revolute joint around pitch Y axis) -->
+    <origin xyz="0.0015 -0.21304 -0.0586" rpy="0 0 0"/>
+  </joint>
+  <!-- Right Rocker (rigidly locked to chassis bearing, leveled with CAD compensation) -->
   <link name="right_rocker">
     <visual>
-      <geometry><box size="0.60 0.05 0.04"/></geometry>
-      <origin xyz="0 0 0" rpy="0 0 0"/>
+      <origin xyz="0 0 0" rpy="0 0 -1.5707963"/>
+      <geometry>
+        <mesh filename="package://meer_description/meshes/right_rocker.STL"/>
+      </geometry>
       <material name="orange"/>
     </visual>
     <collision>
-      <geometry><box size="0.60 0.05 0.04"/></geometry>
-      <origin xyz="0 0 0" rpy="0 0 0"/>
-    </collision>
-    <inertial>
-      <mass value="4.921"/>
-      <origin xyz="0 0 0" rpy="0 0 0"/>
-      <xacro:solid_box_inertia m="4.921" x="0.60" y="0.05" z="0.04"/>
-    </inertial>
-  </link>
-  <joint name="rightrcker" type="revolute">
+      <origin xyz="0.0 0.05 -0.03" rpy="0 0 0"/>
+      <geometry>
+        <box size="0.72 0.05 0.05"/>
+      </geometry>
+    </collision>
+    <inertial>
+      <mass value="4.9215"/>
+      <origin xyz="-0.01799 -0.00746 -0.00770" rpy="0 0 0"/>
+      <inertia
+        ixx="0.022584" ixy="-0.000464" ixz="-0.004731"
+        iyy="0.231464" iyz="-0.000199" izz="0.214960"/>
+    </inertial>
+  </link>
+  <joint name="rightrcker" type="fixed">
     <parent link="right_bearing"/>
     <child link="right_rocker"/>
-    <origin xyz="0 -0.03 0" rpy="0 0 0"/>
-    <axis xyz="0 1 0"/>
-    <limit lower="-0.26" upper="0.26" effort="100" velocity="2.0"/>
-    <dynamics damping="0.5" friction="0.1"/>
-  </joint>
-  <!-- FRW — Front Right Wheel (continuous driven wheel, rolling around Y axis) -->
+    <origin xyz="0 0 0" rpy="0 0.09904 0"/>
+  </joint>
+  <!-- FRW — Front Right Wheel (driven wheel, rolling around Y axis) -->
   <link name="FRW">
     <visual>
-      <geometry><cylinder radius="0.10" length="0.07"/></geometry>
-      <origin xyz="0 0 0" rpy="1.5707963 0 0"/>
+      <origin xyz="0 0 0" rpy="0 0 -1.5707963"/>
+      <geometry>
+        <mesh filename="package://meer_description/meshes/FRW.STL"/>
+      </geometry>
       <material name="black"/>
     </visual>
     <collision>
-      <geometry><cylinder radius="0.10" length="0.07"/></geometry>
-      <origin xyz="0 0 0" rpy="1.5707963 0 0"/>
-    </collision>
-    <inertial>
-      <mass value="1.911"/>
-      <origin xyz="0 0 0" rpy="0 0 0"/>
-      <xacro:solid_cylinder_inertia m="1.911" r="0.10" h="0.07"/>
+      <origin xyz="0 0.0444 0" rpy="1.5707963 0 0"/>
+      <geometry>
+        <cylinder radius="0.1155" length="0.0889"/>
+      </geometry>
+    </collision>
+    <inertial>
+      <mass value="1.9116"/>
+      <origin xyz="-0.00004 0.04682 0.0" rpy="0 0 0"/>
+      <inertia
+        ixx="0.005538" ixy="0.0" ixz="0.0"
+        iyy="0.008143" iyz="0.0" izz="0.005536"/>
     </inertial>
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